File: starbie.kicad_pcb (KiCad board)
At the start: 2 copper layers, 96.5 x 96 mm, 10 parts, among them J1 Conn_01x04_Pin, J2 Conn_01x08_Pin, J3 Conn_01x05_Pin, J4 Conn_01x02_Pin, SW1 SW_Push, SW2 SW_Push, U1 DHT11

Commit message: Update corrected Gerber and drill outputs with latest PCB fixes.
Co-authored-by: Cursor <cursoragent@cursor.com>
Parts:
- moved U1 38.3 mm to (39.5, 168.8)
- moved R1 37.7 mm to (33.5, 168.2)
Connections:
- J4 pad 2: GND -> Net-(J4-Pin_2)
- U2 pad -: unconnected-(U2-Pad-) -> Net-(J4-Pin_2)
- U2 pad 3: /GPI02 -> /JOYSTICK_Y
- U2 pad 4: /GPI03 -> /SDA
- U2 pad 6: /SDA -> /GPI03
- U2 pad 7: /JOYSTICK_Y -> /GPI02
Routing:
- net GND: track 186.9 -> 350.0 mm, vias 0 -> 1
- net /SDA: track 157.4 -> 262.2 mm
- net /JOYSTICK_X: track 154.3 -> 243.3 mm
- net Net-(J4-Pin_2): track 0.00 -> 53.8 mm, vias 0 -> 1
- net /GPI03: track 105.3 -> 157.6 mm
- net /JOYSTICK_Y: track 74.2 -> 96.0 mm
- net /DHT11 DATA: track 158.0 -> 148.6 mm
- net /GPI02: track 132.7 -> 123.9 mm
- net +3.3V: track 235.9 -> 235.2 mm
