File: starbie.kicad_sch (KiCad schematic)
At the start: 9 parts, among them J1 Conn_01x04_Pin, J2 Conn_01x08_Pin, J3 Conn_01x05_Pin, J4 Conn_01x02_Pin, SW1 SW_Push, SW2 SW_Push, U1 DHT11

Commit message: Update Starbie schematic and PCB layout; add BOM CSV export.
Co-authored-by: Cursor <cursoragent@cursor.com>
Parts:
- J3: footprint Connector_PinHeader_2.54mm:PinHeader_1x05_P2.54mm_Vertical -> Connector_PinSocket_2.54mm:PinSocket_1x05_P2.54mm_Vertical
- J4: footprint Connector_PinHeader_2.54mm:PinHeader_1x02_P2.54mm_Vertical -> Connector_JST:JST_PH_S2B-PH-SM4-TB_1x02-1MP_P2.00mm_Horizontal
Changed lines of the file:
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@@
 			)
 		)
-		(property "Footprint" "Connector_PinHeader_2.54mm:PinHeader_1x05_P2.54mm_Vertical"
+		(property "Footprint" "Connector_PinSocket_2.54mm:PinSocket_1x05_P2.54mm_Vertical"
 			(at 16.51 69.85 0)
 			(hide yes)
@@
 			)
 		)
-		(property "Footprint" "Connector_PinHeader_2.54mm:PinHeader_1x02_P2.54mm_Vertical"
+		(property "Footprint" "Connector_JST:JST_PH_S2B-PH-SM4-TB_1x02-1MP_P2.00mm_Horizontal"
 			(at 20.32 118.11 0)
 			(hide yes)

Commit message: Update corrected Gerber and drill outputs with latest PCB fixes.
Co-authored-by: Cursor <cursoragent@cursor.com>
Connections:
- net GND: no longer J4.2 (Pin_2)
- net GPI02: now also U2.7 (PB08_A6_D6_TX); no longer U2.3 (PA10_A2_D2)
- net GPI03: now also U2.6 (PA9_A5_D5_SCL); no longer U2.4 (PA11_A3_D3)
- net JOYSTICK_Y: now also U2.3 (PA10_A2_D2); no longer U2.7 (PB08_A6_D6_TX)
- net SDA: now also U2.4 (PA11_A3_D3); no longer U2.6 (PA9_A5_D5_SCL)
- net at U2.-: now also J4.2 (Pin_2)
- no-connect marks 15 -> 10
Other:
- moved on the sheet: U1
Changed lines of the file:
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@@
 	(paper "A4")
+	(junction
+		(at 55.118 73.66)
+		(diameter 0)
+		(color 0 0 0 0)
+	)
+	(junction
+		(at 74.93 62.23)
+		(diameter 0)
+		(color 0 0 0 0)
+	)
 	(junction
 		(at 60.452 73.66)
@@
 	)
 	(no_connect
-		(at 72.39 104.14)
-	)
-	(no_connect
-		(at 49.53 68.58)
-	)
-	(no_connect
 		(at 72.39 92.71)
 	)
@@
 	)
 	(no_connect
+		(at 72.39 104.14)
+	)
+	(no_connect
 		(at 72.39 96.52)
-	)
-	(no_connect
-		(at 53.34 68.58)
 	)
 	(no_connect
@@
 	)
 	(no_connect
-		(at 93.98 101.6)
-	)
-	(no_connect
 		(at 100.33 82.55)
 	)
-	(no_connect
-		(at 34.29 68.58)
-	)
-	(no_connect
-		(at 38.1 68.58)
+	(wire
+		(pts
+			(xy 15.24 88.9) (xy 22.86 88.9)
+		)
+		(stroke
+			(width 0)
+			(type default)
+		)
 	)
 	(wire
@@
 	(wire
 		(pts
+			(xy 53.34 120.65) (xy 53.34 73.66)
+		)
+		(stroke
+			(width 0)
+			(type default)
+		)
+	)
+	(wire
+		(pts
 			(xy 111.76 69.85) (xy 111.76 71.12)
 		)
@@
 	(wire
 		(pts
+			(xy 74.93 60.96) (xy 74.93 62.23)
+		)
+		(stroke
+			(width 0)
+			(type default)
+		)
+	)
+	(wire
+		(pts
+			(xy 53.34 73.66) (xy 55.118 73.66)
+		)
+		(stroke
+			(width 0)
+			(type default)
+		)
+	)
+	(wire
+		(pts
 			(xy 38.1 59.69) (xy 45.72 59.69)
 		)
@@
 	(wire
 		(pts
+			(xy 74.93 43.18) (xy 74.93 46.99)
+		)
+		(stroke
+			(width 0)
+			(type default)
+		)
+	)
+	(wire
+		(pts
+			(xy 55.118 73.66) (xy 55.88 73.66)
+		)
+		(stroke
+			(width 0)
+			(type default)
+		)
+	)
+	(wire
+		(pts
 			(xy 12.7 83.82) (xy 22.86 83.82)
 		)
@@
 	(wire
 		(pts
+			(xy 74.93 62.23) (xy 74.93 64.77)
+		)
+		(stroke
+			(width 0)
+			(type default)
+		)
+	)
+	(wire
+		(pts
 			(xy 60.96 73.66) (xy 60.452 73.66)
 		)
@@
 	(wire
 		(pts
-			(xy 15.24 88.9) (xy 22.86 88.9)
-		)
-		(stroke
-			(width 0)
-			(type default)
-		)
-	)
-	(wire
-		(pts
 			(xy 76.2 35.56) (xy 81.28 35.56)
 		)
@@
 		)
 	)
-	(label "JOYSTICK_Y"
+	(wire
+		(pts
+			(xy 25.4 120.65) (xy 53.34 120.65)
+		)
+		(stroke
+			(width 0)
+			(type default)
+		)
+	)
+	(label "GPI02"
 		(at 11.43 104.14 0)
 		(effects
@@
 		)
 	)
-	(label "GPI03"
+	(label "SDA"
 		(at 15.24 92.71 0)
 		(effects
@@
 		)
 	)
-	(label "GND"
-		(at 74.93 59.69 0)
-		(effects
-			(font
-				(size 1.27 1.27)
-			)
-			(justify left bottom)
-		)
-	)
 	(label "SCL"
 		(at 15.24 96.52 0)
@@
 	)
 	(label "DHT11 DATA"
-		(at 82.55 52.07 0)
+		(at 82.55 54.61 0)
 		(effects
 			(font
@@
 		)
 	)
+	(label "JOYSTICK_Y"
+		(at 15.24 88.9 0)
+		(effects
+			(font
+				(size 1.27 1.27)
+			)
+			(justify left bottom)
+		)
+	)
 	(label "JOYSTICK_X"
 		(at 21.59 69.85 0)
@@
 		)
 	)
-	(label "SDA"
+	(label "GPI03"
 		(at 15.24 100.33 0)
-		(effects
-			(font
-				(size 1.27 1.27)
-			)
-			(justify left bottom)
-		)
-	)
-	(label "GPI02"
-		(at 15.24 88.9 0)
 		(effects
 			(font
@@
 			)
 			(justify left bottom)
-		)
-	)
-	(symbol
-		(lib_id "power:GND")
-		(at 25.4 120.65 90)
-		(unit 1)
-		(body_style 1)
-		(exclude_from_sim no)
-		(in_bom yes)
-		(on_board yes)
-		(in_pos_files yes)
-		(dnp no)
-		(fields_autoplaced yes)
-		(property "Reference" "#PWR015"
-			(at 31.75 120.65 0)
-			(hide yes)
-			(show_name no)
-			(do_not_autoplace no)
-			(effects
-				(font
-					(size 1.27 1.27)
-				)
-			)
-		)
-		(property "Value" "GND"
-			(at 29.21 120.6499 90)
-			(show_name no)
-			(do_not_autoplace no)
-			(effects
-				(font
-					(size 1.27 1.27)
-				)
-				(justify right)
-			)
-		)
-		(property "Footprint" ""
-			(at 25.4 120.65 0)
-			(hide yes)
-			(show_name no)
-			(do_not_autoplace no)
-			(effects
-				(font
-					(size 1.27 1.27)
-				)
-			)
-		)
-		(property "Datasheet" ""
-			(at 25.4 120.65 0)
-			(hide yes)
-			(show_name no)
-			(do_not_autoplace no)
-			(effects
-				(font
-					(size 1.27 1.27)
-				)
-			)
-		)
-		(property "Description" "Power symbol creates a global label with name \"GND\" , ground"
-			(at 25.4 120.65 0)
-			(hide yes)
-			(show_name no)
-			(do_not_autoplace no)
-			(effects
-				(font
-					(size 1.27 1.27)
-				)
-			)
-		)
-		(pin "1"
-		)
-		(instances
-			(project "starbie"
-				(path "/0317b452-a1b7-45b1-86f0-abd0d959d24f"
-					(reference "#PWR015")
-					(unit 1)
-				)
-			)
 		)
 	)
@@
 	(symbol
 		(lib_id "power:GND")
+		(at 74.93 64.77 0)
+		(unit 1)
+		(body_style 1)
+		(exclude_from_sim no)
+		(in_bom yes)
+		(on_board yes)
+		(in_pos_files yes)
+		(dnp no)
+		(fields_autoplaced yes)
+		(property "Reference" "#PWR017"
+			(at 74.93 71.12 0)
+			(hide yes)
+			(show_name no)
+			(do_not_autoplace no)
+			(effects
+				(font
+					(size 1.27 1.27)
+				)
+			)
+		)
+		(property "Value" "GND"
+			(at 74.93 69.85 0)
+			(show_name no)
+			(do_not_autoplace no)
+			(effects
+				(font
+					(size 1.27 1.27)
+				)
+			)
+		)
+		(property "Footprint" ""
+			(at 74.93 64.77 0)
+			(hide yes)
+			(show_name no)
+			(do_not_autoplace no)
+			(effects
+				(font
+					(size 1.27 1.27)
+				)
+			)
+		)
+		(property "Datasheet" ""
+			(at 74.93 64.77 0)
+			(hide yes)
+			(show_name no)
+			(do_not_autoplace no)
+			(effects
+				(font
+					(size 1.27 1.27)
+				)
+			)
+		)
+		(property "Description" "Power symbol creates a global label with name \"GND\" , ground"
+			(at 74.93 64.77 0)
+			(hide yes)
+			(show_name no)
+			(do_not_autoplace no)
+			(effects
+				(font
+					(size 1.27 1.27)
+				)
+			)
+		)
+		(pin "1"
+		)
+		(instances
+			(project "starbie"
+				(path "/0317b452-a1b7-45b1-86f0-abd0d959d24f"
+					(reference "#PWR017")
+					(unit 1)
+				)
+			)
+		)
+	)
+	(symbol
+		(lib_id "power:GND")
 		(at 55.88 59.69 0)
 		(unit 1)
@@
 	(symbol
 		(lib_id "Sensor:DHT11")
-		(at 74.93 52.07 0)
+		(at 74.93 54.61 0)
 		(unit 1)
 		(body_style 1)
@@
 		(fields_autoplaced yes)
 		(property "Reference" "U1"
-			(at 68.58 50.7999 0)
+			(at 68.58 53.3399 0)
 			(show_name no)
 			(do_not_autoplace no)
@@
 		)
 		(property "Value" "DHT11"
-			(at 68.58 53.3399 0)
+			(at 68.58 55.8799 0)
 			(show_name no)
 			(do_not_autoplace no)
@@
 		)
 		(property "Footprint" "Sensor:Aosong_DHT11_5.5x12.0_P2.54mm"
-			(at 74.93 62.23 0)
+			(at 74.93 64.77 0)
 			(hide yes)
 			(show_name no)
@@
 		)
 		(property "Datasheet" "http://akizukidenshi.com/download/ds/aosong/DHT11.pdf"
-			(at 78.74 45.72 0)
+			(at 78.74 48.26 0)
 			(hide yes)
 			(show_name no)
@@
 		)
 		(property "Description" "3.3V to 5.5V, temperature and humidity module, DHT11"
-			(at 74.93 52.07 0)
+			(at 74.93 54.61 0)
 			(hide yes)
 			(show_name no)
@@
 	(symbol
 		(lib_id "power:+3.3V")
-		(at 74.93 44.45 0)
+		(at 74.93 43.18 0)
 		(unit 1)
 		(body_style 1)
@@
 		(in_pos_files yes)
 		(dnp no)
-		(fields_autoplaced yes)
 		(property "Reference" "#PWR011"
-			(at 74.93 48.26 0)
+			(at 74.93 46.99 0)
 			(hide yes)
 			(show_name no)
@@
 		)
 		(property "Value" "+3.3V"
-			(at 74.93 39.37 0)
+			(at 74.676 40.132 0)
 			(show_name no)
 			(do_not_autoplace no)
@@
 		)
 		(property "Footprint" ""
-			(at 74.93 44.45 0)
+			(at 74.93 43.18 0)
 			(hide yes)
 			(show_name no)
@@
 		)
 		(property "Datasheet" ""
-			(at 74.93 44.45 0)
+			(at 74.93 43.18 0)
 			(hide yes)
 			(show_name no)
@@
 		)
 		(property "Description" "Power symbol creates a global label with name \"+3.3V\""
-			(at 74.93 44.45 0)
-			(hide yes)
-			(show_name no)
+			(at 74.93 43.18 0)
+			(hide yes)
+			(show_name no)
